File: pcb-design.kicad_pcb (KiCad board)
At the start: 2 copper layers, 18.1 x 31.6 mm, 7 parts, among them J1 SM05B-SRSS-TBLFSN, U2 OS102011MA1QS1, U4 MOUDLE-SEEEDUINO-XIAO-ESP32C3

Commit message: update for jlcpcb
Parts:
- removed J1: SM05B-SRSS-TBLFSN, ul_SM05B-SRSS-TB-LF-SN-:CONN5_SM05B-SRSS_JST
- added J2: SM06B-SRSS-TBLFSN, SM06B-SRSS-TB:CONN_SM06B-SRSS-TB_JST, F.Cu at (142.7, 124.5)
- R1, R2: footprint ul_RC0402FR-0710KL:RC0402N_YAG -> RC0402FR-0710KL:RC0402N_YAG
- U2: footprint ul_OS102011MA1QS1:SWITCH_11MA1QS1 -> OS102011MA1QS1:SWITCH_11MA1QS1
- U4: footprint xiao ESP32C3_PCBa:MOUDLE14P-SMD-2.54-21X17.8MM -> MOUDLE-SEEEDUINO-XIAO-ESP32C3-2:MOUDLE14P-SMD-2.54-21X17.8MM
Connections:
- U1 pad 2: Net-(U1--) -> (no net)
- U4 pad 14: unconnected-(U4-5V-Pad14) -> Net-(U4-5V)
Routing:
- net Net-(U4-5V): track 0.00 -> 40.4 mm, vias 0 -> 2
- net Net-(U1-+): track 22.7 -> 4.42 mm, vias 2 -> 0
- net Net-(U1--): track 16.6 -> 0.00 mm, vias 2 -> 0
- net Net-(U4-GND): track 61.0 -> 44.9 mm, vias 3 -> 2
- net Net-(U4-3V3): track 24.8 -> 29.6 mm
- net Net-(U4-PA9_A5_D5_SCL): track 11.7 -> 7.77 mm, vias 0 -> 2
- net Net-(U4-PA8_A4_D4_SDA): track 10.1 -> 8.73 mm
- net Net-(U4-PA6_A10_D10_MOSI): track 27.1 -> 26.6 mm
Other:
- board size 18.1 x 31.6 mm -> 18.5 x 31.6 mm
- board text added: "v4.0.2"
- board text removed: "v4.0.1"
