File: pcb-design.kicad_pcb (KiCad board)
At the start: 2 copper layers, 18.8 x 43.7 mm, 13 parts, among them J1 SM04B-SRSS-TBLFSN, J2 SM04B-SRSS-TBLFSN, U2 OS102011MA1QS1, U3 TSIC206-TO92, U4 MOUDLE-SEEEDUINO-XIAO-ESP32C3

Commit message: v4.0.8 - weer een nieuwe versie aaa
Parts:
- moved R2 1.61 mm to (149.0, 126.0)
- moved R3 1.06 mm to (151.5, 128.0)
Routing:
- net /SW-OUT: track 20.1 -> 21.2 mm
- net /esp-3.3: track 26.6 -> 27.4 mm
- net /D0: track 6.10 -> 6.61 mm
Other:
- outline, holes or cut-outs redrawn
