File: pcb-design.kicad_sch (KiCad schematic)
At the start: 7 parts, among them J1 SM05B-SRSS-TBLFSN, U2 OS102011MA1QS1, U4 MOUDLE-SEEEDUINO-XIAO-ESP32C3

Commit message: v4.0.1
Connections:
- net at U4.1 (PA02_A0_D0): now also U2.3
- net at U4.12 (3V3): now also J1.1; no longer J1.2
- net at U4.13 (GND): now also C1.2, J1.2, R2.1, U2.1
- net at U1.2 (-), U4.15 (-): no longer R2.1
- net at R1.1, U4.16 (+): now also U1.1 (+); no longer U2.1
- net at U2.2: no longer U1.1 (+)
Other:
- moved on the sheet: U2

Commit message: update for jlcpcb
Parts:
- removed J1: SM05B-SRSS-TBLFSN, CONN5_SM05B-SRSS_JST, symbol SM05B-SRSS-TB-LF-SN-:SM05B-SRSS-TBLFSN
- added J2: SM06B-SRSS-TBLFSN, CONN_SM06B-SRSS-TB_JST, symbol SM06B-SRSS-TB:SM06B-SRSS-TBLFSN
Connections:
- net at U4.11 (PA6_A10_D10_MOSI): now also J2.3
- net at U4.12 (3V3): now also J2.1
- net at C1.2, R2.1, U2.1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: now also J2.2
- net at U4.14 (5V): now also J2.6
- net at R1.1, U1.1 (+): no longer U4.16 (+)
- net at U4.5 (PA8_A4_D4_SDA): now also J2.4
- net at U4.6 (PA9_A5_D5_SCL): now also J2.5
Changed lines of the file:
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@@
   (junction (at 48.26 107.95) (diameter 0) (color 0 0 0 0)
   )
-  (junction (at 152.4 107.95) (diameter 0) (color 0 0 0 0)
-  )
   (junction (at 226.06 78.74) (diameter 0) (color 0 0 0 0)
   )
@@
     (stroke (width 0) (type default))
   )
-  (wire (pts (xy 238.76 137.16) (xy 200.66 137.16))
-    (stroke (width 0) (type default))
-  )
-  (wire (pts (xy 181.61 125.73) (xy 181.61 151.13))
-    (stroke (width 0) (type default))
-  )
-  (wire (pts (xy 195.58 99.06) (xy 236.22 99.06))
+  (wire (pts (xy 195.58 99.06) (xy 240.03 99.06))
     (stroke (width 0) (type default))
   )
@@
     (stroke (width 0) (type default))
   )
-  (wire (pts (xy 152.4 86.36) (xy 152.4 107.95))
-    (stroke (width 0) (type default))
-  )
   (wire (pts (xy 124.46 90.17) (xy 124.46 58.42))
     (stroke (width 0) (type default))
   )
-  (wire (pts (xy 212.09 101.6) (xy 236.22 101.6))
-    (stroke (width 0) (type default))
-  )
-  (wire (pts (xy 154.94 107.95) (xy 154.94 125.73))
-    (stroke (width 0) (type default))
-  )
-  (wire (pts (xy 152.4 107.95) (xy 154.94 107.95))
+  (wire (pts (xy 212.09 101.6) (xy 240.03 101.6))
     (stroke (width 0) (type default))
   )
@@
     (stroke (width 0) (type default))
   )
-  (wire (pts (xy 152.4 82.55) (xy 152.4 77.47))
+  (wire (pts (xy 232.41 74.93) (xy 232.41 106.68))
     (stroke (width 0) (type default))
   )
@@
     (stroke (width 0) (type default))
   )
-  (wire (pts (xy 236.22 82.55) (xy 236.22 93.98))
-    (stroke (width 0) (type default))
-  )
-  (wire (pts (xy 152.4 77.47) (xy 163.83 77.47))
-    (stroke (width 0) (type default))
-  )
-  (wire (pts (xy 200.66 137.16) (xy 200.66 151.13))
+  (wire (pts (xy 240.03 82.55) (xy 240.03 93.98))
+    (stroke (width 0) (type default))
+  )
+  (wire (pts (xy 82.55 107.95) (xy 238.76 107.95))
     (stroke (width 0) (type default))
   )
@@
     (stroke (width 0) (type default))
   )
-  (wire (pts (xy 163.83 77.47) (xy 163.83 120.65))
-    (stroke (width 0) (type default))
-  )
   (wire (pts (xy 124.46 58.42) (xy 212.09 58.42))
     (stroke (width 0) (type default))
   )
-  (wire (pts (xy 163.83 120.65) (xy 190.5 120.65))
-    (stroke (width 0) (type default))
-  )
-  (wire (pts (xy 236.22 104.14) (xy 205.74 104.14))
+  (wire (pts (xy 240.03 104.14) (xy 205.74 104.14))
     (stroke (width 0) (type default))
   )
@@
     (stroke (width 0) (type default))
   )
-  (wire (pts (xy 181.61 125.73) (xy 154.94 125.73))
-    (stroke (width 0) (type default))
-  )
-  (wire (pts (xy 238.76 142.24) (xy 190.5 142.24))
+  (wire (pts (xy 185.42 74.93) (xy 232.41 74.93))
     (stroke (width 0) (type default))
   )
@@
     (stroke (width 0) (type default))
   )
-  (wire (pts (xy 181.61 151.13) (xy 200.66 151.13))
-    (stroke (width 0) (type default))
-  )
   (wire (pts (xy 205.74 104.14) (xy 205.74 63.5))
     (stroke (width 0) (type default))
@@
     (stroke (width 0) (type default))
   )
-  (wire (pts (xy 190.5 120.65) (xy 190.5 142.24))
-    (stroke (width 0) (type default))
-  )
   (wire (pts (xy 110.49 81.28) (xy 110.49 74.93))
     (stroke (width 0) (type default))
@@
     (stroke (width 0) (type default))
   )
+  (wire (pts (xy 238.76 107.95) (xy 238.76 137.16))
+    (stroke (width 0) (type default))
+  )
   (wire (pts (xy 62.23 81.28) (xy 110.49 81.28))
     (stroke (width 0) (type default))
   )
-  (wire (pts (xy 236.22 96.52) (xy 226.06 96.52))
+  (wire (pts (xy 232.41 106.68) (xy 240.03 106.68))
+    (stroke (width 0) (type default))
+  )
+  (wire (pts (xy 240.03 96.52) (xy 226.06 96.52))
     (stroke (width 0) (type default))
   )
@@
     (stroke (width 0) (type default))
   )
-  (wire (pts (xy 82.55 107.95) (xy 152.4 107.95))
-    (stroke (width 0) (type default))
-  )
   (wire (pts (xy 48.26 86.36) (xy 135.89 86.36))
     (stroke (width 0) (type default))
@@
     (stroke (width 0) (type default))
   )
-  (wire (pts (xy 185.42 82.55) (xy 236.22 82.55))
+  (wire (pts (xy 185.42 82.55) (xy 240.03 82.55))
     (stroke (width 0) (type default))
   )
@@
     (pin "4")
     (pin "12")
-    (pin "15")
     (pin "8")
     (pin "14")
@@
     (pin "7")
     (pin "1")
-    (pin "16")
     (pin "2")
     (instances
@@
     )
   )
-  (symbol (lib_id "2023-11-23_19-25-58:RC0402FR-0710KL") (at 69.85 142.24 0) (unit 1)
+  (symbol (lib_name "RC0402FR-0710KL_1") (lib_id "2023-11-23_19-25-58:RC0402FR-0710KL") (at 69.85 142.24 0) (unit 1)
     (in_bom yes) (on_board yes) (dnp no) (fields_autoplaced)
     (property "Reference" "R2" (at 76.2 135.89 0)
@@
       (effects (font (size 1.27 1.27)) hide)
     )
-    (pin "1")
-    (pin "2")
+    (pin "")
+    (pin "1")
     (instances
       (project "pcb-design"
@@
     )
   )
-  (symbol (lib_id "SM05B-SRSS-TB-LF-SN-:SM05B-SRSS-TBLFSN") (at 236.22 93.98 0) (unit 1)
-    (in_bom yes) (on_board yes) (dnp no) (fields_autoplaced)
-    (property "Reference" "J1" (at 250.19 97.79 0)
+  (symbol (lib_id "2023-11-23_19-58-11:OS102011MA1QS1") (at 102.87 72.39 180) (unit 1)
+    (in_bom yes) (on_board yes) (dnp no) (fields_autoplaced)
+    (property "Reference" "U2" (at 82.55 59.69 0)
+      (effects (font (size 1.524 1.524)))
+    )
+    (property "Value" "OS102011MA1QS1" (at 82.55 62.23 0)
+      (effects (font (size 1.524 1.524)))
+    )
+    (property "Footprint" "SWITCH_11MA1QS1" (at 102.87 72.39 0)
+      (effects (font (size 1.27 1.27) italic) hide)
+    )
+    (property "Datasheet" "OS102011MA1QS1" (at 102.87 72.39 0)
+      (effects (font (size 1.27 1.27) italic) hide)
+    )
+    (pin "2")
+    (pin "1")
+    (pin "3")
+    (instances
+      (project "pcb-design"
+        (path "/5f569c9b-d86b-422c-aa8b-ae82a353c125"
+          (reference "U2") (unit 1)
+        )
+      )
+    )
+  )
+  (symbol (lib_id "2023-11-23_19-25-58:RC0402FR-0710KL") (at 69.85 107.95 0) (unit 1)
+    (in_bom yes) (on_board yes) (dnp no) (fields_autoplaced)
+    (property "Reference" "R1" (at 76.2 101.6 0)
+      (effects (font (size 1.524 1.524)))
+    )
+    (property "Value" "RC0402FR-0710KL" (at 76.2 104.14 0)
+      (effects (font (size 1.524 1.524)))
+    )
+    (property "Footprint" "RC0402N_YAG" (at 69.85 107.95 0)
+      (effects (font (size 1.27 1.27) italic) hide)
+    )
+    (property "Datasheet" "RC0402FR-0710KL" (at 69.85 107.95 0)
+      (effects (font (size 1.27 1.27) italic) hide)
+    )
+    (pin "2")
+    (pin "1")
+    (instances
+      (project "pcb-design"
+        (path "/5f569c9b-d86b-422c-aa8b-ae82a353c125"
+          (reference "R1") (unit 1)
+        )
+      )
+    )
+  )
+  (symbol (lib_id "SM06B-SRSS-TB:SM06B-SRSS-TBLFSN") (at 240.03 93.98 0) (unit 1)
+    (in_bom yes) (on_board yes) (dnp no) (fields_autoplaced)
+    (property "Reference" "J2" (at 254 99.06 0)
       (effects (font (size 1.524 1.524)) (justify left))
     )
-    (property "Value" "SM05B-SRSS-TBLFSN" (at 250.19 100.33 0)
+    (property "Value" "SM06B-SRSS-TBLFSN" (at 254 101.6 0)
       (effects (font (size 1.524 1.524)) (justify left))
     )
-    (property "Footprint" "CONN5_SM05B-SRSS_JST" (at 236.22 93.98 0)
-      (effects (font (size 1.27 1.27) italic) hide)
-    )
-    (property "Datasheet" "SM05B-SRSS-TBLFSN" (at 236.22 93.98 0)
-      (effects (font (size 1.27 1.27) italic) hide)
-    )
+    (property "Footprint" "CONN_SM06B-SRSS-TB_JST" (at 240.03 93.98 0)
+      (effects (font (size 1.27 1.27) italic) hide)
+    )
+    (property "Datasheet" "SM06B-SRSS-TBLFSN" (at 240.03 93.98 0)
+      (effects (font (size 1.27 1.27) italic) hide)
+    )
+    (pin "2")
     (pin "3")
-    (pin "2")
+    (pin "4")
+    (pin "1")
+    (pin "6")
     (pin "5")
-    (pin "1")
-    (pin "4")
-    (instances
-      (project "pcb-design"
-        (path "/5f569c9b-d86b-422c-aa8b-ae82a353c125"
-          (reference "J1") (unit 1)
-        )
-      )
-    )
-  )
-  (symbol (lib_id "2023-11-23_19-58-11:OS102011MA1QS1") (at 102.87 72.39 180) (unit 1)
-    (in_bom yes) (on_board yes) (dnp no) (fields_autoplaced)
-    (property "Reference" "U2" (at 82.55 59.69 0)
-      (effects (font (size 1.524 1.524)))
-    )
-    (property "Value" "OS102011MA1QS1" (at 82.55 62.23 0)
-      (effects (font (size 1.524 1.524)))
-    )
-    (property "Footprint" "SWITCH_11MA1QS1" (at 102.87 72.39 0)
-      (effects (font (size 1.27 1.27) italic) hide)
-    )
-    (property "Datasheet" "OS102011MA1QS1" (at 102.87 72.39 0)
-      (effects (font (size 1.27 1.27) italic) hide)
-    )
-    (pin "2")
-    (pin "1")
-    (pin "3")
-    (instances
-      (project "pcb-design"
-        (path "/5f569c9b-d86b-422c-aa8b-ae82a353c125"
-          (reference "U2") (unit 1)
-        )
-      )
-    )
-  )
-  (symbol (lib_id "2023-11-23_19-25-58:RC0402FR-0710KL") (at 69.85 107.95 0) (unit 1)
-    (in_bom yes) (on_board yes) (dnp no) (fields_autoplaced)
-    (property "Reference" "R1" (at 76.2 101.6 0)
-      (effects (font (size 1.524 1.524)))
-    )
-    (property "Value" "RC0402FR-0710KL" (at 76.2 104.14 0)
-      (effects (font (size 1.524 1.524)))
-    )
-    (property "Footprint" "RC0402N_YAG" (at 69.85 107.95 0)
-      (effects (font (size 1.27 1.27) italic) hide)
-    )
-    (property "Datasheet" "RC0402FR-0710KL" (at 69.85 107.95 0)
-      (effects (font (size 1.27 1.27) italic) hide)
-    )
-    (pin "2")
-    (pin "1")
-    (instances
-      (project "pcb-design"
-        (path "/5f569c9b-d86b-422c-aa8b-ae82a353c125"
-          (reference "R1") (unit 1)
-        )
-      )
+    (instances
+      (project "pcb-design"
+        (path "/5f569c9b-d86b-422c-aa8b-ae82a353c125"
+          (reference "J2") (unit 1)
+        )
+      )
