File: v4.1/v4.0.10c.kicad_sch (KiCad schematic)
At the start: 12 parts, among them J1 SM04B-SRSS-TBLFSN, J2 SM04B-SRSS-TBLFSN, U2 OS102011MA1QS1, U3 TSIC206-TO92, U4 MOUDLE-SEEEDUINO-XIAO-ESP32C3

Commit message: updated LED footprint for JLCPCB
Parts:
- U3: now not fitted
Changed lines of the file:
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@@
 		(in_bom yes)
 		(on_board yes)
-		(dnp no)
+		(dnp yes)
 		(property "Reference" "U3"
 			(at 154.94 37.338 0)

Commit message: prepare U2 hand assembly and source XIAO
Parts:
- U2: now not fitted
Changed lines of the file:
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@@
 		(in_bom yes)
 		(on_board yes)
-		(dnp no)
+		(dnp yes)
 		(property "Reference" "U2"
 			(at 227.838 65.786 0)
